File: mollusc_motion_board/DynamixelConnection.kicad_sch (KiCad schematic)
At the start: 8 parts, among them U3 SN74AHCT125N, U7 74LVC2G241

Commit message: Board v2 wip
Parts:
- C1: value 0.1uF 16V -> 0.1uF 50V; footprint HangOn_Mainboard:R0603 -> molluscmotion:C0603
- R10, R11, R12, R13: footprint HangOn_Mainboard:R0603 -> molluscmotion:R0603
- U3: footprint HangOn_Mainboard:SOIC-14_L8.7-W3.9-P1.27-LS6.0-BL -> molluscmotion:SOIC-14_L8.7-W3.9-P1.27-LS6.0-BL
- U7: footprint HangOn_Mainboard:SSOP-8_L3.0-W2.8-P0.65-LS4.0-BL -> molluscmotion:SSOP-8_L3.0-W2.8-P0.65-LS4.0-BL
Changed lines of the file:
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@@
       (effects (font (size 1.27 1.27)))
     )
-    (property "Footprint" "HangOn_Mainboard:SSOP-8_L3.0-W2.8-P0.65-LS4.0-BL" (at 151.13 91.44 0)
+    (property "Footprint" "molluscmotion:SSOP-8_L3.0-W2.8-P0.65-LS4.0-BL" (at 151.13 91.44 0)
       (effects (font (size 1.27 1.27)) hide)
     )
@@
       (effects (font (size 1.27 1.27)))
     )
-    (property "Footprint" "HangOn_Mainboard:SSOP-8_L3.0-W2.8-P0.65-LS4.0-BL" (at 148.59 110.49 0)
+    (property "Footprint" "molluscmotion:SSOP-8_L3.0-W2.8-P0.65-LS4.0-BL" (at 148.59 110.49 0)
       (effects (font (size 1.27 1.27)) hide)
     )
@@
       (effects (font (size 1.27 1.27)) (justify left))
     )
-    (property "Footprint" "HangOn_Mainboard:R0603" (at 97.282 93.98 90)
+    (property "Footprint" "molluscmotion:R0603" (at 97.282 93.98 90)
       (effects (font (size 1.27 1.27)) hide)
     )
@@
       (effects (font (size 1.27 1.27)) (justify left))
     )
-    (property "Value" "0.1uF 16V " (at 68.58 74.93 90)
-      (effects (font (size 1.27 1.27)) (justify left))
-    )
-    (property "Footprint" "HangOn_Mainboard:R0603" (at 69.85 77.7748 0)
+    (property "Value" "0.1uF 50V " (at 68.58 74.93 90)
+      (effects (font (size 1.27 1.27)) (justify left))
+    )
+    (property "Footprint" "molluscmotion:C0603" (at 69.85 77.7748 0)
       (effects (font (size 1.27 1.27)) hide)
     )
@@
       (effects (font (size 1.27 1.27)) (justify left))
     )
-    (property "Footprint" "HangOn_Mainboard:R0603" (at 121.412 93.98 90)
+    (property "Footprint" "molluscmotion:R0603" (at 121.412 93.98 90)
       (effects (font (size 1.27 1.27)) hide)
     )
@@
       (effects (font (size 1.27 1.27)) (justify left))
     )
-    (property "Value" "0.1uF 16V " (at 236.22 91.44 90)
-      (effects (font (size 1.27 1.27)) (justify left))
-    )
-    (property "Footprint" "HangOn_Mainboard:R0603" (at 237.49 94.2848 0)
+    (property "Value" "0.1uF 50V " (at 236.22 91.44 90)
+      (effects (font (size 1.27 1.27)) (justify left))
+    )
+    (property "Footprint" "molluscmotion:C0603" (at 237.49 94.2848 0)
       (effects (font (size 1.27 1.27)) hide)
     )
@@
       (effects (font (size 1.524 1.524)) (justify left))
     )
-    (property "Footprint" "HangOn_Mainboard:SOIC-14_L8.7-W3.9-P1.27-LS6.0-BL" (at 74.93 100.33 0)
+    (property "Footprint" "molluscmotion:SOIC-14_L8.7-W3.9-P1.27-LS6.0-BL" (at 74.93 100.33 0)
       (effects (font (size 1.524 1.524)) (justify left) hide)
     )
@@
       (effects (font (size 1.27 1.27)) (justify left))
     )
-    (property "Footprint" "HangOn_Mainboard:R0603" (at 170.688 87.63 90)
+    (property "Footprint" "molluscmotion:R0603" (at 170.688 87.63 90)
       (effects (font (size 1.27 1.27)) hide)
     )
@@
       (effects (font (size 1.27 1.27)) (justify left))
     )
-    (property "Footprint" "HangOn_Mainboard:R0603" (at 170.688 77.47 90)
+    (property "Footprint" "molluscmotion:R0603" (at 170.688 77.47 90)
       (effects (font (size 1.27 1.27)) hide)
     )
@@
       (effects (font (size 1.27 1.27)) (justify left))
     )
-    (property "Footprint" "HangOn_Mainboard:SSOP-8_L3.0-W2.8-P0.65-LS4.0-BL" (at 237.49 107.95 0)
-      (effects (font (size 1.27 1.27)) hide)
-    )
+    (property "Footprint" "molluscmotion:SSOP-8_L3.0-W2.8-P0.65-LS4.0-BL" (at 237.49 107.95 0)
+      (effects (font (size 1.27 1.27)) hide)
+    )

Commit message: PCB v1.2 Layout
Other:
- moved on the sheet: C1, U7C
Changed lines of the file:
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@@
   (junction (at 123.19 100.33) (diameter 0) (color 0 0 0 0)
   )
-  (junction (at 237.49 95.25) (diameter 0) (color 0 0 0 0)
+  (junction (at 224.79 -41.91) (diameter 0) (color 0 0 0 0)
   )
   (junction (at 99.06 100.33) (diameter 0) (color 0 0 0 0)
@@
     (stroke (width 0) (type default))
   )
-  (wire (pts (xy 237.49 88.9) (xy 237.49 95.25))
+  (wire (pts (xy 224.79 -48.26) (xy 224.79 -41.91))
     (stroke (width 0) (type default))
   )
@@
     (stroke (width 0) (type default))
   )
-  (wire (pts (xy 120.65 100.33) (xy 123.19 100.33))
+  (wire (pts (xy 118.11 100.33) (xy 123.19 100.33))
     (stroke (width 0) (type default))
   )
@@
     (stroke (width 0) (type default))
   )
-  (wire (pts (xy 120.65 100.33) (xy 120.65 106.68))
-    (stroke (width 0) (type default))
-  )
   (wire (pts (xy 59.69 100.33) (xy 43.18 100.33))
     (stroke (width 0) (type default))
@@
     (stroke (width 0) (type default))
   )
-  (wire (pts (xy 237.49 95.25) (xy 237.49 97.79))
+  (wire (pts (xy 224.79 -41.91) (xy 224.79 -39.37))
     (stroke (width 0) (type default))
   )
@@
     (stroke (width 0) (type default))
   )
-  (wire (pts (xy 224.79 95.25) (xy 229.87 95.25))
+  (wire (pts (xy 212.09 -41.91) (xy 217.17 -41.91))
     (stroke (width 0) (type default))
   )
@@
     (effects (font (size 1.27 1.27)) (justify right bottom))
   )
-  (text "DYNAMIXEL_CONNECTION" (at 92.71 41.91 0)
+  (text "DYNAMIXEL_CONNECTION" (at 88.9 -27.94 0)
     (effects (font (size 5.08 5.08)) (justify left bottom))
   )
@@
     (effects (font (size 1.27 1.27)) (justify left bottom))
   )
-  (hierarchical_label "DYN_DATA" (shape bidirectional) (at 120.65 106.68 270) (fields_autoplaced)
+  (hierarchical_label "DYN_DATA" (shape bidirectional) (at 118.11 100.33 180) (fields_autoplaced)
     (effects (font (size 1.27 1.27)) (justify right))
   )
@@
     )
   )
-  (symbol (lib_id "power:GND") (at 237.49 118.11 0) (unit 1)
+  (symbol (lib_id "power:GND") (at 224.79 -19.05 0) (unit 1)
     (in_bom yes) (on_board yes) (dnp no) (fields_autoplaced)
-    (property "Reference" "#PWR024" (at 237.49 124.46 0)
-      (effects (font (size 1.27 1.27)) hide)
-    )
-    (property "Value" "GND" (at 237.49 123.19 0)
-      (effects (font (size 1.27 1.27)))
-    )
-    (property "Footprint" "" (at 237.49 118.11 0)
-      (effects (font (size 1.27 1.27)) hide)
-    )
-    (property "Datasheet" "" (at 237.49 118.11 0)
+    (property "Reference" "#PWR024" (at 224.79 -12.7 0)
+      (effects (font (size 1.27 1.27)) hide)
+    )
+    (property "Value" "GND" (at 224.79 -13.97 0)
+      (effects (font (size 1.27 1.27)))
+    )
+    (property "Footprint" "" (at 224.79 -19.05 0)
+      (effects (font (size 1.27 1.27)) hide)
+    )
+    (property "Datasheet" "" (at 224.79 -19.05 0)
       (effects (font (size 1.27 1.27)) hide)
     )
@@
     )
   )
-  (symbol (lib_id "Device:C") (at 233.68 95.25 90) (unit 1)
-    (in_bom yes) (on_board yes) (dnp no)
-    (property "Reference" "C1" (at 232.41 96.52 90)
-      (effects (font (size 1.27 1.27)) (justify left))
-    )
-    (property "Value" "0.1uF 50V " (at 236.22 91.44 90)
-      (effects (font (size 1.27 1.27)) (justify left))
-    )
-    (property "Footprint" "molluscmotion:C0603" (at 237.49 94.2848 0)
-      (effects (font (size 1.27 1.27)) hide)
-    )
-    (property "Datasheet" "~" (at 233.68 95.25 0)
-      (effects (font (size 1.27 1.27)) hide)
-    )
-    (property "Comment" "place near 74LVC2G241" (at 250.19 93.98 90)
-      (effects (font (size 1.27 1.27)))
-    )
-    (property "JLCPCB Part #" "C14663" (at 233.68 95.25 0)
+  (symbol (lib_id "Device:C") (at 220.98 -41.91 90) (unit 1)
+    (in_bom yes) (on_board yes) (dnp no)
+    (property "Reference" "C1" (at 219.71 -40.64 90)
+      (effects (font (size 1.27 1.27)) (justify left))
+    )
+    (property "Value" "0.1uF 50V " (at 223.52 -45.72 90)
+      (effects (font (size 1.27 1.27)) (justify left))
+    )
+    (property "Footprint" "molluscmotion:C0603" (at 224.79 -42.8752 0)
+      (effects (font (size 1.27 1.27)) hide)
+    )
+    (property "Datasheet" "~" (at 220.98 -41.91 0)
+      (effects (font (size 1.27 1.27)) hide)
+    )
+    (property "Comment" "place near 74LVC2G241" (at 237.49 -43.18 90)
+      (effects (font (size 1.27 1.27)))
+    )
+    (property "JLCPCB Part #" "C14663" (at 220.98 -41.91 0)
       (effects (font (size 1.27 1.27)) hide)
     )
@@
     )
   )
-  (symbol (lib_id "power:GND") (at 224.79 95.25 270) (unit 1)
-    (in_bom yes) (on_board yes) (dnp no)
-    (property "Reference" "#PWR01" (at 218.44 95.25 0)
-      (effects (font (size 1.27 1.27)) hide)
-    )
-    (property "Value" "GND" (at 222.25 95.25 90)
+  (symbol (lib_id "power:GND") (at 212.09 -41.91 270) (unit 1)
+    (in_bom yes) (on_board yes) (dnp no)
+    (property "Reference" "#PWR01" (at 205.74 -41.91 0)
+      (effects (font (size 1.27 1.27)) hide)
+    )
+    (property "Value" "GND" (at 209.55 -41.91 90)
       (effects (font (size 1.27 1.27)) (justify right))
     )
-    (property "Footprint" "" (at 224.79 95.25 0)
-      (effects (font (size 1.27 1.27)) hide)
-    )
-    (property "Datasheet" "" (at 224.79 95.25 0)
+    (property "Footprint" "" (at 212.09 -41.91 0)
+      (effects (font (size 1.27 1.27)) hide)
+    )
+    (property "Datasheet" "" (at 212.09 -41.91 0)
       (effects (font (size 1.27 1.27)) hide)
     )
@@
     )
   )
-  (symbol (lib_id "power:+5V") (at 237.49 88.9 0) (unit 1)
-    (in_bom yes) (on_board yes) (dnp no)
-    (property "Reference" "#PWR05" (at 237.49 92.71 0)
-      (effects (font (size 1.27 1.27)) hide)
-    )
-    (property "Value" "+5V" (at 232.41 87.63 0)
-      (effects (font (size 1.27 1.27)) (justify left))
-    )
-    (property "Footprint" "" (at 237.49 88.9 0)
-      (effects (font (size 1.27 1.27)) hide)
-    )
-    (property "Datasheet" "" (at 237.49 88.9 0)
+  (symbol (lib_id "power:+5V") (at 224.79 -48.26 0) (unit 1)
+    (in_bom yes) (on_board yes) (dnp no)
+    (property "Reference" "#PWR05" (at 224.79 -44.45 0)
+      (effects (font (size 1.27 1.27)) hide)
+    )
+    (property "Value" "+5V" (at 219.71 -49.53 0)
+      (effects (font (size 1.27 1.27)) (justify left))
+    )
+    (property "Footprint" "" (at 224.79 -48.26 0)
+      (effects (font (size 1.27 1.27)) hide)
+    )
+    (property "Datasheet" "" (at 224.79 -48.26 0)
       (effects (font (size 1.27 1.27)) hide)
     )
@@
     )
   )
-  (symbol (lib_id "74xGxx:74LVC2G241") (at 237.49 107.95 0) (unit 3)
+  (symbol (lib_id "74xGxx:74LVC2G241") (at 224.79 -29.21 0) (unit 3)
     (in_bom yes) (on_board yes) (dnp no) (fields_autoplaced)
-    (property "Reference" "U7" (at 243.84 106.68 0)
-      (effects (font (size 1.27 1.27)) (justify left))
-    )
-    (property "Value" "74LVC2G241" (at 243.84 109.22 0)
-      (effects (font (size 1.27 1.27)) (justify left))
-    )
-    (property "Footprint" "molluscmotion:SSOP-8_L3.0-W2.8-P0.65-LS4.0-BL" (at 237.49 107.95 0)
-      (effects (font (size 1.27 1.27)) hide)
-    )
-    (property "Datasheet" "http://www.ti.com/lit/sg/scyt129e/scyt129e.pdf" (at 237.49 107.95 0)
-      (effects (font (size 1.27 1.27)) hide)
-    )
-    (property "JLCPCB Part #" "C2676069" (at 237.49 107.95 0)
-      (effects (font (size 1.27 1.27)) hide)
-    )
+    (property "Reference" "U7" (at 231.14 -30.48 0)
+      (effects (font (size 1.27 1.27)) (justify left))
+    )
+    (property "Value" "74LVC2G241" (at 231.14 -27.94 0)
+      (effects (font (size 1.27 1.27)) (justify left))
+    )
+    (property "Footprint" "molluscmotion:SSOP-8_L3.0-W2.8-P0.65-LS4.0-BL" (at 224.79 -29.21 0)
+      (effects (font (size 1.27 1.27)) hide)
+    )
+    (property "Datasheet" "http://www.ti.com/lit/sg/scyt129e/scyt129e.pdf" (at 224.79 -29.21 0)
+      (effects (font (size 1.27 1.27)) hide)
+    )
+    (property "JLCPCB Part #" "C2676069" (at 224.79 -29.21 0)
+      (effects (font (size 1.27 1.27)) hide)
+    )
