File: mollusc_motion_board/mollusc_motion_board.kicad_pcb (KiCad board)
At the start: 4 copper layers, 120 x 120 mm, 67 parts, among them J1 Neopixel Conn., J2 Barrel_Jack_Switch 12V, J3 RJ45_LED_Shielded, J4 RJ45 x4, J5 Conn_01x06_Pin, J6 D36V50F5, J7 Endswitches Test Conn, SW1 SW_Push, SW2 SW_Push, U1 SN74AHCT125N, U2 SN74AHCT125N, U3 SN74AHCT125N, U4 74HC14, U6 SN74AHCT125N, U7 74LVC2G241, U9 Teensy4.1

Commit message: PCB v1.2
v1.2, produced by JLCPCB
Parts:
- removed SW1, SW2: SW_Push, molluscmotion:KEY-SMD_4P-L6.1-W6.1-P4.50-LS9.0
- added CB1: CircuitBreaker_1P_closed, clockdiv:CircuitBreaker_0603_closed, F.Cu at (162.7, 99.6)
- added CB2: CircuitBreaker_1P_closed, clockdiv:CircuitBreaker_0603_closed, F.Cu at (155.6, 99.6)
- added H5: MountingHole, MountingHole:MountingHole_3.2mm_M3_DIN965_Pad, F.Cu at (184.5, 76.6)
- added H6: MountingHole, MountingHole:MountingHole_3.2mm_M3_DIN965_Pad, F.Cu at (184.5, 121.6)
- added J8: NP Power, Connector_PinHeader_2.54mm:PinHeader_1x02_P2.54mm_Vertical, F.Cu at (110.6, 113.1)
- added TP_END_S1: TestPoint, TestPoint:TestPoint_THTPad_1.5x1.5mm_Drill0.7mm, F.Cu at (116.6, 100.3)
- added TP_END_S2: TestPoint, TestPoint:TestPoint_THTPad_1.5x1.5mm_Drill0.7mm, F.Cu at (116.6, 97.8)
- added TP_END_S3: TestPoint, TestPoint:TestPoint_THTPad_1.5x1.5mm_Drill0.7mm, F.Cu at (116.6, 95.2)
- added U5: TSA063G60-250, molluscmotion:KEY-SMD_4P-L6.1-W6.1-P4.50-LS9.0, F.Cu at (99.7, 146.4)
- added U8: TSA063G60-250, molluscmotion:KEY-SMD_4P-L6.1-W6.1-P4.50-LS9.0, F.Cu at (82.1, 129.1)
- D3: value SMAJ14A_C908768 -> SMAJ14A
- H1, H2, H3, H4: footprint MountingHole:MountingHole_3.2mm_M3_DIN965_Pad_TopBottom -> MountingHole:MountingHole_3.2mm_M3_DIN965_Pad
- J1: value Neopixel Conn. -> NP Power+Sig
- J7: value Endswitches Test Conn -> NP Power; footprint Connector_PinHeader_2.54mm:PinHeader_1x03_P2.54mm_Vertical -> Connector_PinHeader_2.54mm:PinHeader_1x02_P2.54mm_Vertical
- moved H3 217.3 mm to (152.0, 154.1)
- moved H2 188.8 mm to (107.0, 154.1)
- moved H4 141.3 mm to (74.5, 121.6)
- moved H1 125.9 mm to (74.5, 76.6)
- moved J7 17.9 mm to (108.0, 115.8), turned to 45 degrees
- moved J1 5.06 mm to (105.2, 118.6), turned to 45 degrees
- moved R14 4.03 mm to (112.0, 119.9), turned to 45 degrees
- moved TP4 2.98 mm to (116.2, 122.4)
- moved C9 0.38 mm to (93.3, 64.3)
Connections:
- H1 pad 1: (no net) -> GND
- H2 pad 1: (no net) -> GND
- H4 pad 1: (no net) -> GND
- J1 pad 1: GND -> +5V
- J1 pad 2: Net-(J1-Pin_2) -> GND
- J1 pad 3: +5V -> Net-(J1-Pin_3)
- J4 pad A6: +12V -> GND
- J7 pad 1: /STEPPER_01_END -> +5V
- J7 pad 2: /STEPPER_02_END -> GND
- R1 pad 2: GND -> Net-(CB2-Pad2)
- R14 pad 1: Net-(J1-Pin_2) -> Net-(J1-Pin_3)
- R15 pad 2: GND -> Net-(CB1-Pad2)
Routing:
- net +12V: track 50.6 -> 100.1 mm
- net +5V: track 368.9 -> 405.2 mm, vias 9 -> 11
- net /BAT+: track 80.6 -> 88.9 mm
- net +3.3V: track 257.2 -> 260.8 mm, vias 6 -> 11
- net Net-(J1-Pin_3): track 0.00 -> 3.46 mm
- net /NEOPIXEL_SIG: track 30.6 -> 27.2 mm
- net Net-(J1-Pin_2): track 3.08 -> 0.00 mm
- net Net-(CB2-Pad2): track 0.00 -> 2.63 mm
- net Net-(CB1-Pad2): track 0.00 -> 2.62 mm
- net GND: track 45.7 -> 44.2 mm, vias 7 -> 101
- net Net-(U9-16_A2_RX4_SCL1): track 46.8 -> 45.3 mm
- net /DynamixelConnection/DYN_DATA: track 16.7 -> 18.0 mm
- net /BAT-: track 82.9 -> 81.6 mm
- net Net-(U9-17_A3_TX4_SDA1): track 28.7 -> 29.9 mm
- added copper zone on B.Cu, net +12V
Other:
- board text added: "5V GND SIG"
- board text added: "cut and replace with resistor to dim the led"
- board text added: "red"
- board text removed: "12V"
